File: PCB/FREEBOARD.kicad_sch (KiCad schematic)
At the start: 0 parts

Commit message: Key Matrix & LEDs
Parts:
- added A1: RaspberryPi_Pico, Module:RaspberryPi_Pico_Common_Unspecified, symbol MCU_Module:RaspberryPi_Pico
- added D1, D10, D11, D12, D13, D14, D15, D16, D17, D18, D19, D2, D20, D21, D22, D23, D24, D25, D26, D27, D28, D29, D3, D30, D31, D32, D33, D34, D35, D36, D37, D38, D39, D4, D40, D41, D42, D43, D44, D45, D46, D47, D48, D49, D5, D50, D51, D52, D53, D54, D55, D56, D57, D58, D59, D6, D60, D61, D62, D63, D64, D65, D66, D67, D68, D69, D7, D70, D71, D72, D73, D74, D75, D76, D77, D78, D79, D8, D80, D81, D9: 1N4148, Diode_THT:D_DO-35_SOD27_P7.62mm_Horizontal, symbol Diode:1N4148
- added D100, D101, D102, D103, D104, D105, D106, D107, D108, D109, D110, D111, D112, D113, D114, D115, D116, D117, D118, D119, D120, D121, D122, D123, D124, D125, D126, D127, D128, D129, D130, D131, D132, D133, D134, D135, D136, D137, D138, D139, D140, D141, D142, D143, D144, D145, D146, D147, D148, D149, D150, D151, D152, D153, D154, D155, D156, D157, D158, D159, D160, D161, D162, D163, D82, D83, D84, D85, D86, D87, D88, D89, D90, D91, D92, D93, D94, D95, D96, D97, D98, D99: SK6812MINI-E, footprints:SK6812MINI-E_fixed, symbol SK6812MINI-E:SK6812MINI-E
- added J1: OLED_DISPLAY, footprints:SSD1306-0.91-OLED-4pin-128x32, symbol Connector_Generic:Conn_01x04
- added S1: MX_stab, PCM_marbastlib-mx:STAB_MX_P_6.25u, symbol PCM_marbastlib-mx:MX_stab
- added SW1, SW10, SW11, SW12, SW13, SW14, SW15, SW16, SW17, SW18, SW19, SW2, SW20, SW21, SW22, SW23, SW24, SW25, SW26, SW27, SW28, SW29, SW3, SW30, SW31, SW32, SW33, SW34, SW35, SW36, SW37, SW38, SW39, SW4, SW40, SW41, SW42, SW43, SW44, SW45, SW46, SW47, SW48, SW49, SW5, SW50, SW51, SW52, SW53, SW54, SW55, SW56, SW57, SW58, SW59, SW6, SW60, SW61, SW62, SW63, SW64, SW65, SW66, SW67, SW68, SW69, SW7, SW70, SW71, SW72, SW73, SW74, SW75, SW76, SW77, SW78, SW79, SW8, SW80, SW81, SW9: SW_Push_45deg, symbol Switch:SW_Push_45deg
- added SW82: RotaryEncoder_Switch, Rotary_Encoder:RotaryEncoder_Alps_EC11E-Switch_Vertical_H20mm, symbol RotaryEncoder_Switch:RotaryEncoder_Switch
Connections:
- new net: SW10.1, SW25.1, SW40.1, SW54.1, SW68.1, SW77.1
- new net: D10.2 (A), SW10.2
- new net: SW11.1, SW26.1, SW41.1, SW55.1, SW69.1, SW78.1
- new net: D41.2 (A), SW41.2
- new net: D130.2 (DOUT), D133.4 (DIN)
- new net: SW21.1, SW36.1, SW50.1, SW6.1, SW64.1
- new net: D6.2 (A), SW6.2
- new net: SW14.1, SW29.1, SW44.1, SW58.1, SW72.1, SW81.1
- new net: D44.2 (A), SW44.2
- new net: D72.2 (A), SW72.2
- new net: D11.2 (A), SW11.2
- new net: D54.2 (A), SW54.2
- new net: D45.1 (K), D46.1 (K), D47.1 (K), D48.1 (K), D49.1 (K), D50.1 (K), D51.1 (K), D52.1 (K), D53.1 (K), D54.1 (K), D55.1 (K), D56.1 (K), D57.1 (K), D58.1 (K), SW24.1, SW39.1, SW53.1, SW67.1, SW9.1
- new net: D50.2 (A), SW50.2
- new net: SW22.1, SW37.1, SW51.1, SW65.1, SW7.1
- new net: D51.2 (A), SW51.2
- new net: D94.2 (DOUT), D95.4 (DIN)
- new net: D93.2 (DOUT), D94.4 (DIN)
- new net: SW23.1, SW38.1, SW52.1, SW66.1, SW8.1
- new net: D52.2 (A), SW52.2
- new net: SW12.1, SW27.1, SW42.1, SW56.1, SW70.1, SW79.1
- new net: D70.2 (A), SW70.2
- new net: SW18.1, SW3.1, SW33.1, SW76.1
- new net: D76.2 (A), SW76.2
- new net: SW16.1, SW31.1, SW46.1, SW60.1, SW74.1
- new net: D31.2 (A), SW31.2
- new net: SW13.1, SW28.1, SW43.1, SW57.1, SW71.1, SW80.1
- new net: D80.2 (A), SW80.2
- new net: D18.2 (A), SW18.2
- new net: D15.1 (K), D16.1 (K), D17.1 (K), D18.1 (K), D19.1 (K), D20.1 (K), D21.1 (K), D22.1 (K), D23.1 (K), D24.1 (K), D25.1 (K), D26.1 (K), D27.1 (K), D28.1 (K), D29.1 (K)
- new net: D20.2 (A), SW20.2
- new net: D53.2 (A), SW53.2
- new net: D104.2 (DOUT), D105.4 (DIN)
- new net: D103.2 (DOUT), D104.4 (DIN)
- new net: SW19.1, SW34.1, SW4.1, SW48.1, SW62.1
- new net: D62.2 (A), SW62.2
- new net: D107.2 (DOUT), D108.4 (DIN)
- new net: D106.2 (DOUT), D107.4 (DIN)
- new net: D141.2 (DOUT), D144.4 (DIN)
- new net: D138.2 (DOUT), D141.4 (DIN)
- new net: D30.1 (K), D31.1 (K), D32.1 (K), D33.1 (K), D34.1 (K), D35.1 (K), D36.1 (K), D37.1 (K), D38.1 (K), D39.1 (K), D40.1 (K), D41.1 (K), D42.1 (K), D43.1 (K), D44.1 (K)
- new net: D40.2 (A), SW40.2
- new net: D1.1 (K), D10.1 (K), D11.1 (K), D12.1 (K), D13.1 (K), D14.1 (K), D2.1 (K), D3.1 (K), D4.1 (K), D5.1 (K), D6.1 (K), D7.1 (K), D8.1 (K), D9.1 (K)
- new net: D147.2 (DOUT), D150.4 (DIN)
- new net: D144.2 (DOUT), D147.4 (DIN)
- new net: D77.2 (A), SW77.2
- new net: D91.2 (DOUT), D92.4 (DIN)
- new net: D45.2 (A), SW45.2
- new net: SW17.1, SW2.1, SW32.1, SW47.1, SW61.1, SW75.1
- new net: D2.2 (A), SW2.2
- new net: D89.2 (DOUT), D90.4 (DIN)
- new net: D33.2 (A), SW33.2
- new net: D42.2 (A), SW42.2
- new net: D157.2 (DOUT), D160.4 (DIN)
- new net: D154.2 (DOUT), D157.4 (DIN)
- new net: D37.2 (A), SW37.2
- new net: D14.2 (A), SW14.2
- new net: D142.2 (DOUT), D145.4 (DIN)
- new net: D139.2 (DOUT), D142.4 (DIN)
- new net: D59.1 (K), D60.1 (K), D61.1 (K), D62.1 (K), D63.1 (K), D64.1 (K), D65.1 (K), D66.1 (K), D67.1 (K), D68.1 (K), D69.1 (K), D70.1 (K), D71.1 (K), D72.1 (K)
- new net: D69.2 (A), SW69.2
- new net: D58.2 (A), SW58.2
- new net: D96.2 (DOUT), D97.4 (DIN)
- new net: D95.2 (DOUT), D96.4 (DIN)
- new net: D23.2 (A), SW23.2
- new net: D19.2 (A), SW19.2
- new net: D86.2 (DOUT), D87.4 (DIN)
- new net: D85.2 (DOUT), D86.4 (DIN)
- new net: D9.2 (A), SW9.2
- new net: D81.2 (A), SW81.2
- new net: D74.2 (A), SW74.2
- new net: D68.2 (A), SW68.2
- new net: D158.2 (DOUT), D161.4 (DIN)
- new net: D15.2 (A), SW15.2
- new net: D38.2 (A), SW38.2
- new net: D59.2 (A), SW59.2
- new net: D75.2 (A), SW75.2
- new net: D150.2 (DOUT), D153.4 (DIN)
- new net: D26.2 (A), SW26.2
- new net: SW20.1, SW35.1, SW49.1, SW5.1, SW63.1
- new net: D92.2 (DOUT), D93.4 (DIN)
- new net: D12.2 (A), SW12.2
- new net: D43.2 (A), SW43.2
- new net: D35.2 (A), SW35.2
- new net: D73.1 (K), D74.1 (K), D75.1 (K), D76.1 (K), D77.1 (K), D78.1 (K), D79.1 (K), D80.1 (K), D81.1 (K)
- new net: D65.2 (A), SW65.2
- new net: D48.2 (A), SW48.2
- new net: D78.2 (A), SW78.2
- new net: D97.2 (DOUT), D98.4 (DIN)
- new net: D60.2 (A), SW60.2
- new net: D117.2 (DOUT), D120.4 (DIN)
- new net: D114.2 (DOUT), D117.4 (DIN)
- new net: D148.2 (DOUT), D151.4 (DIN)
- new net: D145.2 (DOUT), D148.4 (DIN)
- new net: D125.2 (DOUT), D128.4 (DIN)
- new net: D122.2 (DOUT), D125.4 (DIN)
- new net: D112.2 (DOUT), D115.4 (DIN)
- new net: D109.2 (DOUT), D112.4 (DIN)
- new net: D34.2 (A), SW34.2
- new net: D67.2 (A), SW67.2
- new net: D137.2 (DOUT), D140.4 (DIN)
- new net: D16.2 (A), SW16.2
- new net: D83.2 (DOUT), D84.4 (DIN)
- new net: D82.2 (DOUT), D83.4 (DIN)
- new net: D13.2 (A), SW13.2
- new net: D132.2 (DOUT), D135.4 (DIN)
- new net: D129.2 (DOUT), D132.4 (DIN)
- new net: D136.2 (DOUT), D139.4 (DIN)
- new net: D5.2 (A), SW5.2
- new net: D162.2 (DOUT), D163.4 (DIN)
- new net: D152.2 (DOUT), D155.4 (DIN)
- new net: D149.2 (DOUT), D152.4 (DIN)
- new net: A1.13 (GND), A1.18 (GND), A1.23 (GND), A1.28 (GND), A1.3 (GND), A1.38 (GND), A1.8 (GND)
- new net: D63.2 (A), SW63.2
- new net: D84.2 (DOUT), D85.4 (DIN)
- new net: D113.2 (DOUT), D116.4 (DIN)
- new net: D110.2 (DOUT), D113.4 (DIN)
- new net: D22.2 (A), SW22.2
- new net: D56.2 (A), SW56.2
- new net: D49.2 (A), SW49.2
- new net: D47.2 (A), SW47.2
- new net: D3.2 (A), SW3.2
- new net: D159.2 (DOUT), D162.4 (DIN)
- new net: D55.2 (A), SW55.2
- new net: D98.2 (DOUT), D99.4 (DIN)
- new net: D146.2 (DOUT), D149.4 (DIN)
- new net: D143.2 (DOUT), D146.4 (DIN)
- new net: D29.2 (A), SW29.2
- new net: D111.2 (DOUT), D114.4 (DIN)
- new net: D66.2 (A), SW66.2
- new net: D115.2 (DOUT), D118.4 (DIN)
- new net: D39.2 (A), SW39.2
- new net: D124.2 (DOUT), D127.4 (DIN)
- new net: D121.2 (DOUT), D124.4 (DIN)
- new net: D71.2 (A), SW71.2
- new net: D8.2 (A), SW8.2
- new net: D151.2 (DOUT), D154.4 (DIN)
- new net: D30.2 (A), SW30.2
- new net: D105.2 (DOUT), D106.4 (DIN)
- new net: SW1.1, SW15.1, SW30.1, SW45.1, SW59.1, SW73.1
- new net: D1.2 (A), SW1.2
- new net: D153.2 (DOUT), D156.4 (DIN)
- new net: D25.2 (A), SW25.2
- new net: D119.2 (DOUT), D122.4 (DIN)
- new net: D79.2 (A), SW79.2
- new net: D46.2 (A), SW46.2
- new net: D100.2 (DOUT), D101.4 (DIN)
- new net: D21.2 (A), SW21.2
- new net: D17.2 (A), SW17.2
- new net: D102.2 (DOUT), D103.4 (DIN)
- new net: D101.2 (DOUT), D102.4 (DIN)
- new net: D24.2 (A), SW24.2
- new net: D4.2 (A), SW4.2
- new net: D36.2 (A), SW36.2
- new net: D128.2 (DOUT), D131.4 (DIN)
- new net: D28.2 (A), SW28.2
- new net: D27.2 (A), SW27.2
- new net: D116.2 (DOUT), D119.4 (DIN)
- new net: D88.2 (DOUT), D89.4 (DIN)
- new net: D118.2 (DOUT), D121.4 (DIN)
- new net: D140.2 (DOUT), D143.4 (DIN)
- new net: D127.2 (DOUT), D130.4 (DIN)
- new net: D73.2 (A), SW73.2
- new net: D123.2 (DOUT), D126.4 (DIN)
- new net: D120.2 (DOUT), D123.4 (DIN)
- new net: D126.2 (DOUT), D129.4 (DIN)
- new net: D61.2 (A), SW61.2
- new net: D64.2 (A), SW64.2
- new net: D32.2 (A), SW32.2
- new net: D57.2 (A), SW57.2
- new net: D155.2 (DOUT), D158.4 (DIN)
- new net: D156.2 (DOUT), D159.4 (DIN)
- new net: D87.2 (DOUT), D88.4 (DIN)
- new net: D7.2 (A), SW7.2
- new net: D131.2 (DOUT), D134.4 (DIN)
- new net +5V: D100.1 (VDD), D101.1 (VDD), D102.1 (VDD), D103.1 (VDD), D104.1 (VDD), D105.1 (VDD), D106.1 (VDD), D107.1 (VDD), D108.1 (VDD), D109.1 (VDD), D110.1 (VDD), D111.1 (VDD), D112.1 (VDD), D113.1 (VDD), D114.1 (VDD), D115.1 (VDD), D116.1 (VDD), D117.1 (VDD), D118.1 (VDD), D119.1 (VDD), D120.1 (VDD), D121.1 (VDD), D122.1 (VDD), D123.1 (VDD), D124.1 (VDD), D125.1 (VDD), D126.1 (VDD), D127.1 (VDD), D128.1 (VDD), D129.1 (VDD), D130.1 (VDD), D131.1 (VDD), D132.1 (VDD), D133.1 (VDD), D134.1 (VDD), D135.1 (VDD), D136.1 (VDD), D137.1 (VDD), D138.1 (VDD), D139.1 (VDD), D140.1 (VDD), D141.1 (VDD), D142.1 (VDD), D143.1 (VDD), D144.1 (VDD), D145.1 (VDD), D146.1 (VDD), D147.1 (VDD), D148.1 (VDD), D149.1 (VDD), D150.1 (VDD), D151.1 (VDD), D152.1 (VDD), D153.1 (VDD), D154.1 (VDD), D155.1 (VDD), D156.1 (VDD), D157.1 (VDD), D158.1 (VDD), D159.1 (VDD), D160.1 (VDD), D161.1 (VDD), D162.1 (VDD), D163.1 (VDD), D82.1 (VDD), D83.1 (VDD), D84.1 (VDD), D85.1 (VDD), D86.1 (VDD), D87.1 (VDD), D88.1 (VDD), D89.1 (VDD), D90.1 (VDD), D91.1 (VDD), D92.1 (VDD), D93.1 (VDD), D94.1 (VDD), D95.1 (VDD), D96.1 (VDD), D97.1 (VDD), D98.1 (VDD), D99.1 (VDD)
- new net GND: D100.3 (VSS), D101.3 (VSS), D102.3 (VSS), D103.3 (VSS), D104.3 (VSS), D105.3 (VSS), D106.3 (VSS), D107.3 (VSS), D108.3 (VSS), D109.3 (VSS), D110.3 (VSS), D111.3 (VSS), D112.3 (VSS), D113.3 (VSS), D114.3 (VSS), D115.3 (VSS), D116.3 (VSS), D117.3 (VSS), D118.3 (VSS), D119.3 (VSS), D120.3 (VSS), D121.3 (VSS), D122.3 (VSS), D123.3 (VSS), D124.3 (VSS), D125.3 (VSS), D126.3 (VSS), D127.3 (VSS), D128.3 (VSS), D129.3 (VSS), D130.3 (VSS), D131.3 (VSS), D132.3 (VSS), D133.3 (VSS), D134.3 (VSS), D135.3 (VSS), D136.3 (VSS), D137.3 (VSS), D138.3 (VSS), D139.3 (VSS), D140.3 (VSS), D141.3 (VSS), D142.3 (VSS), D143.3 (VSS), D144.3 (VSS), D145.3 (VSS), D146.3 (VSS), D147.3 (VSS), D148.3 (VSS), D149.3 (VSS), D150.3 (VSS), D151.3 (VSS), D152.3 (VSS), D153.3 (VSS), D154.3 (VSS), D155.3 (VSS), D156.3 (VSS), D157.3 (VSS), D158.3 (VSS), D159.3 (VSS), D160.3 (VSS), D161.3 (VSS), D162.3 (VSS), D163.3 (VSS), D82.3 (VSS), D83.3 (VSS), D84.3 (VSS), D85.3 (VSS), D86.3 (VSS), D87.3 (VSS), D88.3 (VSS), D89.3 (VSS), D90.3 (VSS), D91.3 (VSS), D92.3 (VSS), D93.3 (VSS), D94.3 (VSS), D95.3 (VSS), D96.3 (VSS), D97.3 (VSS), D98.3 (VSS), D99.3 (VSS)
- new net RGB: D82.4 (DIN)

Commit message: PCB update
Parts:
- added D164: SK6812MINI-E, footprints:SK6812MINI-E_fixed, symbol SK6812MINI-E:SK6812MINI-E
Connections:
- net +5V: now also D164.1 (VDD)
- net GND: now also D164.3 (VSS)
- net at D163.2 (DOUT): now also D164.4 (DIN)
Changed lines of the file:
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@@
 	)
 	(junction
+		(at 309.88 218.44)
+		(diameter 0)
+		(color 0 0 0 0)
+	)
+	(junction
 		(at 36.83 52.07)
 		(diameter 0)
@@
 	)
 	(junction
+		(at 309.88 233.68)
+		(diameter 0)
+		(color 0 0 0 0)
+	)
+	(junction
 		(at 194.31 73.66)
 		(diameter 0)
@@
 	(wire
 		(pts
+			(xy 309.88 218.44) (xy 326.39 218.44)
+		)
+		(stroke
+			(width 0)
+			(type default)
+		)
+	)
+	(wire
+		(pts
 			(xy 218.44 153.67) (xy 219.71 153.67)
 		)
@@
 	(wire
 		(pts
+			(xy 317.5 226.06) (xy 318.77 226.06)
+		)
+		(stroke
+			(width 0)
+			(type default)
+		)
+	)
+	(wire
+		(pts
 			(xy 161.29 64.77) (xy 153.67 64.77)
 		)
@@
 	(wire
 		(pts
+			(xy 309.88 233.68) (xy 326.39 233.68)
+		)
+		(stroke
+			(width 0)
+			(type default)
+		)
+	)
+	(wire
+		(pts
 			(xy 34.29 50.8) (xy 41.91 50.8)
 		)
@@
 					(unit 1)
 				)
+			)
+		)
+	)
+	(symbol
+		(lib_id "SK6812MINI-E:SK6812MINI-E")
+		(at 326.39 226.06 0)
+		(unit 1)
+		(body_style 1)
+		(exclude_from_sim no)
+		(in_bom yes)
+		(on_board yes)
+		(in_pos_files yes)
+		(dnp no)
+		(property "Reference" "D164"
+			(at 335.28 214.8839 0)
+			(show_name no)
+			(do_not_autoplace no)
+			(effects
+				(font
+					(size 1.27 1.27)
+				)
+			)
+		)
+		(property "Value" "SK6812MINI-E"
+			(at 335.28 217.424 0)
+			(show_name no)
+			(do_not_autoplace no)
+			(effects
+				(font
+					(size 1.27 1.27)
+					(thickness 0.254)
+					(bold yes)
+				)
+			)
+		)
+		(property "Footprint" "footprints:SK6812MINI-E_fixed"
+			(at 327.66 233.68 0)
+			(hide yes)
+			(show_name no)
+			(do_not_autoplace no)
+			(effects
+				(font
+					(size 1.27 1.27)
+				)
+				(justify left top)
+			)
+		)
+		(property "Datasheet" "https://cdn-shop.adafruit.com/product-files/4960/4960_SK6812MINI-E_REV02_EN.pdf"
+			(at 328.93 235.585 0)
+			(hide yes)
+			(show_name no)
+			(do_not_autoplace no)
+			(effects
+				(font
+					(size 1.27 1.27)
+				)
+				(justify left top)
+			)
+		)
+		(property "Description" "RGB LED with integrated controller"
+			(at 326.39 226.06 0)
+			(hide yes)
+			(show_name no)
+			(do_not_autoplace no)
+			(effects
+				(font
+					(size 1.27 1.27)
+				)
+			)
+		)
+		(pin "2"
+		)
+		(pin "4"
+		)
+		(pin "3"
+		)
+		(pin "1"
+		)
+		(instances
+			(project "FREEBOARD"
+				(path "/08dde3a1-be10-42d5-942d-cd142127e9fa"
+					(reference "D164")
+					(unit 1)
+				)

Commit message: Finished RGB LEDs
Parts:
- added D165, D166, D167, D168, D169, D170, D171, D172, D173: SK6812MINI-E, footprints:SK6812MINI-E_fixed, symbol SK6812MINI-E:SK6812MINI-E
- added D174: 1N4148, Diode_THT:D_DO-35_SOD27_P7.62mm_Horizontal, symbol Diode:1N4148
Connections:
- net +5V: now also D165.1 (VDD), D166.1 (VDD), D167.1 (VDD), D168.1 (VDD), D169.1 (VDD), D170.1 (VDD), D171.1 (VDD), D172.1 (VDD), D173.1 (VDD)
- net GND: now also J1.4 (Pin_4), SW82.C, D165.3 (VSS), D166.3 (VSS), D167.3 (VSS), D168.3 (VSS), D169.3 (VSS), D170.3 (VSS), D171.3 (VSS), D172.3 (VSS), D173.3 (VSS)
- net RGB: now also A1.27 (GPIO21)
- net Col10: now reaches SW10.1, SW25.1, SW40.1, SW54.1, SW68.1, SW77.1
- net Col10: now also A1.21 (GPIO16)
- net Col11: now reaches SW11.1, SW26.1, SW41.1, SW55.1, SW69.1, SW78.1
- net Col11: now also A1.22 (GPIO17)
- net Col6: now reaches SW21.1, SW36.1, SW50.1, SW6.1, SW64.1
- net Col6: now also A1.16 (GPIO12)
- net Col14: now reaches SW14.1, SW29.1, SW44.1, SW58.1, SW72.1, SW81.1
- net Col14: now also A1.26 (GPIO20), SW82.S2
- net Col9: now reaches D45.1 (K), D46.1 (K), D47.1 (K), D48.1 (K), D49.1 (K), D50.1 (K), D51.1 (K), D52.1 (K), D53.1 (K), D54.1 (K), D55.1 (K), D56.1 (K), D57.1 (K), D58.1 (K), SW24.1, SW39.1, SW53.1, SW67.1, SW9.1
- net Col9: now also A1.20 (GPIO15), A1.5 (GPIO3)
- net Col7: now reaches SW22.1, SW37.1, SW51.1, SW65.1, SW7.1
- net Col7: now also A1.17 (GPIO13)
- net Col8: now reaches SW23.1, SW38.1, SW52.1, SW66.1, SW8.1
- net Col8: now also A1.19 (GPIO14)
- net Col12: now reaches SW12.1, SW27.1, SW42.1, SW56.1, SW70.1, SW79.1
- net Col12: now also A1.24 (GPIO18)
- net Col3: now reaches SW18.1, SW3.1, SW33.1, SW76.1
- net Col3: now also A1.12 (GPIO9)
- net Col1: now reaches SW16.1, SW31.1, SW46.1, SW60.1, SW74.1
- net Col1: now also A1.10 (GPIO7)
- net Col13: now reaches SW13.1, SW28.1, SW43.1, SW57.1, SW71.1, SW80.1
- net Col13: now also A1.25 (GPIO19)
- net Row1: now reaches D15.1 (K), D16.1 (K), D17.1 (K), D18.1 (K), D19.1 (K), D20.1 (K), D21.1 (K), D22.1 (K), D23.1 (K), D24.1 (K), D25.1 (K), D26.1 (K), D27.1 (K), D28.1 (K), D29.1 (K)
- net Row1: now also A1.2 (GPIO1)
- net Col4: now reaches SW19.1, SW34.1, SW4.1, SW48.1, SW62.1
- net Col4: now also A1.14 (GPIO10)
- net Row2: now reaches D30.1 (K), D31.1 (K), D32.1 (K), D33.1 (K), D34.1 (K), D35.1 (K), D36.1 (K), D37.1 (K), D38.1 (K), D39.1 (K), D40.1 (K), D41.1 (K), D42.1 (K), D43.1 (K), D44.1 (K)
- net Row2: now also A1.4 (GPIO2)
- net Row0: now reaches D1.1 (K), D10.1 (K), D11.1 (K), D12.1 (K), D13.1 (K), D14.1 (K), D2.1 (K), D3.1 (K), D4.1 (K), D5.1 (K), D6.1 (K), D7.1 (K), D8.1 (K), D9.1 (K)
- net Row0: now also A1.1 (GPIO0), D174.1 (K)
- net at D91.4 (DIN): now also D90.2 (DOUT)
- net Col2: now reaches SW17.1, SW2.1, SW32.1, SW47.1, SW61.1, SW75.1
- net Col2: now also A1.11 (GPIO8)
- net Row4: now reaches D59.1 (K), D60.1 (K), D61.1 (K), D62.1 (K), D63.1 (K), D64.1 (K), D65.1 (K), D66.1 (K), D67.1 (K), D68.1 (K), D69.1 (K), D70.1 (K), D71.1 (K), D72.1 (K)
- net Row4: now also A1.6 (GPIO4)
- net at D161.2 (DOUT): now also D138.4 (DIN)
- net Col5: now reaches SW20.1, SW35.1, SW49.1, SW5.1, SW63.1
- net Col5: now also A1.15 (GPIO11)
- net Row5: now reaches D73.1 (K), D74.1 (K), D75.1 (K), D76.1 (K), D77.1 (K), D78.1 (K), D79.1 (K), D80.1 (K), D81.1 (K)
- net Row5: now also A1.7 (GPIO5)
- net at D137.4 (DIN): now also D160.2 (DOUT)
- net OLED_SDA: now reaches A1.29 (GPIO22)
- net OLED_SDA: now also J1.1 (Pin_1)
- net OLED_SCL: now reaches A1.31 (GPIO26_ADC0)
- net OLED_SCL: now also J1.2 (Pin_2)
- net ENC_A: now reaches A1.32 (GPIO27_ADC1)
- net ENC_A: now also SW82.A
- net ENC_B: now reaches A1.34 (GPIO28_ADC2)
- net ENC_B: now also SW82.B
- net Col0: now reaches A1.9 (GPIO6)
- net Col0: now also SW1.1, SW15.1, SW30.1, SW45.1, SW59.1, SW73.1
- net at D108.2 (DOUT): now also D109.4 (DIN)
- net at D135.2 (DOUT): now also D136.4 (DIN)
- net at D99.2 (DOUT): now also D100.4 (DIN)
- net ESW_A: now reaches SW82.S1
- net ESW_A: now also D174.2 (A)
- net at D164.2 (DOUT): now also D165.4 (DIN)
- net at D111.4 (DIN): now also D134.2 (DOUT)
- new net: D167.2 (DOUT), D168.4 (DIN)
- new net: D166.2 (DOUT), D167.4 (DIN)
- new net: D170.2 (DOUT), D171.4 (DIN)
- new net: D169.2 (DOUT), D170.4 (DIN)
- new net: D172.2 (DOUT), D173.4 (DIN)
- new net: D171.2 (DOUT), D172.4 (DIN)
- new net: D165.2 (DOUT), D166.4 (DIN)
- new net: D168.2 (DOUT), D169.4 (DIN)
- no-connect marks 0 -> 1
Other:
- moved on the sheet: D1, D10, D100, D101, D102, D103, D104, D105, D106, D107, D108, D109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

Commit message: Schematic Update
Parts:
- removed D174: 1N4148, Diode_THT:D_DO-35_SOD27_P7.62mm_Horizontal, symbol Diode:1N4148
- removed SW82: RotaryEncoder_Switch, Rotary_Encoder:RotaryEncoder_Alps_EC11E-Switch_Vertical_H20mm, symbol RotaryEncoder_Switch:RotaryEncoder_Switch
- added C1, C2: 0.1uF, symbol Device:C
- added C10, C11, C12, C13, C14, C15, C16, C17, C18, C19, C20, C21, C22, C23, C24, C25, C26, C27, C28, C29, C30, C31, C32, C33, C34, C35, C36, C37, C38, C39, C4, C40, C41, C42, C43, C44, C45, C46, C47, C48, C49, C50, C51, C52, C53, C54, C55, C56, C57, C58, C59, C6, C60, C61, C62, C63, C64, C65, C66, C67, C68, C69, C7, C70, C71, C72, C73, C74, C75, C76, C77, C78, C79, C8, C80, C81, C82, C83, C84, C85, C86, C87, C88, C89, C9, C90, C91, C92, C93, C94, C95, C96: 100nF, symbol Device:C
- added C3: 10uF, symbol Device:C
- added C5: 470uF, symbol Device:C
- added H1, H2, H3, H4, H5, H6, H7, H8: MountingHole, symbol Mechanical:MountingHole
- added R1: 10k, symbol Device:R
- added R2, R3: 4.7k, symbol Device:R
- added R4: 330, symbol Device:R
- added S2, S3, S4: MX_stab, PCM_marbastlib-mx:STAB_MX_P_6.25u, symbol PCM_marbastlib-mx:MX_stab
- added SW82: RotaryEncoder_Switch, symbol Device:RotaryEncoder_Switch
- added U1: MCP23017x-x-SP, Package_DIP:DIP-28_W7.62mm, symbol Interface_Expansion:MCP23017x-x-SP
- A1: footprint Module:RaspberryPi_Pico_Common_Unspecified -> Module:RaspberryPi_Pico_Common_THT
- J1: footprint footprints:SSD1306-0.91-OLED-4pin-128x32 -> KiCad-SSD1306-0.91-OLED-4pin-128x32.pretty-master:SSD1306-0.91-OLED-4pin-128x32
- renumbered D112 to D110, D115 to D111, D118 to D112, D121 to D113, D124 to D114, D127 to D115, D130 to D116, D133 to D117, D110 to D118, D113 to D119, D116 to D120, D119 to D121, D125 to D123, D128 to D124, D131 to D125, D134 to D126, D111 to D127, D114 to D128, D117 to D129, D120 to D130, D123 to D131, D126 to D132, D129 to D133, D132 to D134
Connections:
- net +5V: now also A1.40 (VBUS), J1.3 (Pin_3), C10.1, C11.1, C12.1, C13.1, C14.1, C15.1, C16.1, C17.1, C18.1, C19.1, C20.1, C21.1, C22.1, C23.1, C24.1, C25.1, C26.1, C27.1, C28.1, C29.1, C30.1, C31.1, C32.1, C33.1, C34.1, C35.1, C36.1, C37.1, C38.1, C39.1, C4.1, C40.1, C41.1, C42.1, C43.1, C44.1, C45.1, C46.1, C47.1, C48.1, C49.1, C5.1, C50.1, C51.1, C52.1, C53.1, C54.1, C55.1, C56.1, C57.1, C58.1, C59.1, C6.1, C60.1, C61.1, C62.1, C63.1, C64.1, C65.1, C66.1, C67.1, C68.1, C69.1, C7.1, C70.1, C71.1, C72.1, C73.1, C74.1, C75.1, C76.1, C77.1, C78.1, C79.1, C8.1, C80.1, C81.1, C82.1, C83.1, C84.1, C85.1, C86.1, C87.1, C88.1, C89.1, C9.1, C90.1, C91.1, C92.1, C93.1, C94.1, C95.1, C96.1
- net Col9: no longer A1.5 (GPIO3), D45.1 (K), D46.1 (K), D47.1 (K), D48.1 (K), D49.1 (K), D50.1 (K), D51.1 (K), D52.1 (K), D53.1 (K), D54.1 (K), D55.1 (K), D56.1 (K), D57.1 (K), D58.1 (K)
- net ENC_A: now also SW82.B, U1.21 (GPA0); no longer A1.32 (GPIO27_ADC1)
- net ENC_B: now also SW82.A, U1.22 (GPA1); no longer A1.34 (GPIO28_ADC2)
- net GND: now also A1.13 (GND), A1.18 (GND), A1.23 (GND), A1.28 (GND), A1.3 (GND), A1.38 (GND), A1.8 (GND), C1.2, C10.2, C11.2, C12.2, C13.2, C14.2, C15.2, C16.2, C17.2, C18.2, C19.2, C2.2, C20.2, C21.2, C22.2, C23.2, C24.2, C25.2, C26.2, C27.2, C28.2, C29.2, C3.2, C30.2, C31.2, C32.2, C33.2, C34.2, C35.2, C36.2, C37.2, C38.2, C39.2, C4.2, C40.2, C41.2, C42.2, C43.2, C44.2, C45.2, C46.2, C47.2, C48.2, C49.2, C5.2, C50.2, C51.2, C52.2, C53.2, C54.2, C55.2, C56.2, C57.2, C58.2, C59.2, C6.2, C60.2, C61.2, C62.2, C63.2, C64.2, C65.2, C66.2, C67.2, C68.2, C69.2, C7.2, C70.2, C71.2, C72.2, C73.2, C74.2, C75.2, C76.2, C77.2, C78.2, C79.2, C8.2, C80.2, C81.2, C82.2, C83.2, C84.2, C85.2, C86.2, C87.2, C88.2, C89.2, C9.2, C90.2, C91.2, C92.2, C93.2, C94.2, C95.2, C96.2, SW82.C, SW82.S1, U1.10 (V_{SS}), U1.15 (A0), U1.16 (A1), U1.17 (A2)
- net OLED_SCL: now also R3.1, U1.12 (SCK)
- net OLED_SDA: now also R2.1, U1.13 (SDA)
- net RGB: now also R4.1; no longer D82.4 (DIN)
- net at D117.2 (DOUT): now also D118.4 (DIN)
- net +3V3: now reaches A1.36 (3V3)
- net +3V3: now also C1.1, C2.1, C3.1, R1.2, R2.2, R3.2, U1.9 (V_{DD})
- new net: D82.4 (DIN), R4.2
- new net: R1.1, U1.18 (~{RESET})
- new net ESW: SW82.S2, U1.23 (GPA2)
- new net Row3: A1.5 (GPIO3), D45.1 (K), D46.1 (K), D47.1 (K), D48.1 (K), D49.1 (K), D50.1 (K), D51.1 (K), D52.1 (K), D53.1 (K), D54.1 (K), D55.1 (K), D56.1 (K), D57.1 (K), D58.1 (K)
- no-connect marks 1 -> 23
Other:
- note added: "CAPSLCK"
- note added: "CONTROLLERS"
- note added: "DECOUPLING"
- note added: "DISPLAY & ENCODER"
- note added: "ENTER"
- note added: "HOLES"
- note added: "KEY MATRIX"
- note added: "LSHIFT"
- note added: "RGB BACKLIGHT"
- note added: "SPACE"
- title: (none) -> FREEBOARD
- moved on the sheet: A1, D1, D10, D100, D101, D102, D103, D104, D105, D106, D107, D108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

Commit message: Finished Schematic
Parts:
- C1, C10, C11, C12, C13, C14, C15, C16, C17, C18, C19, C2, C20, C21, C22, C23, C24, C25, C26, C27, C28, C29, C30, C31, C32, C33, C34, C35, C36, C37, C38, C39, C4, C40, C41, C42, C43, C44, C45, C46, C47, C48, C49, C50, C51, C52, C53, C54, C55, C56, C57, C58, C59, C6, C60, C61, C62, C63, C64, C65, C66, C67, C68, C69, C7, C70, C71, C72, C73, C74, C75, C76, C77, C78, C79, C8, C80, C81, C82, C83, C84, C85, C86, C87, C88, C89, C9, C90, C91, C92, C93, C94, C95, C96: footprint (none) -> Capacitor_SMD:C_0603_1608Metric_Pad1.08x0.95mm_HandSolder
- C3: footprint (none) -> Capacitor_SMD:C_0805_2012Metric_Pad1.18x1.45mm_HandSolder
- C5: footprint (none) -> Capacitor_Tantalum_SMD:CP_EIA-7343-31_Kemet-D_HandSolder
- H1, H2, H3, H4, H5, H6, H7, H8: footprint (none) -> MountingHole:MountingHole_3.2mm_M3
- R1, R2, R3: footprint (none) -> Resistor_SMD:R_0603_1608Metric_Pad0.98x0.95mm_HandSolder
- R4: value 330 -> 510; footprint (none) -> Resistor_SMD:R_0603_1608Metric_Pad0.98x0.95mm_HandSolder
- S1: footprint PCM_marbastlib-mx:STAB_MX_P_6.25u -> PCM_marbastlib-mx:STAB_MX_2u
- S2, S3: footprint PCM_marbastlib-mx:STAB_MX_P_6.25u -> PCM_marbastlib-mx:STAB_MX_2.25u
- S4: footprint PCM_marbastlib-mx:STAB_MX_P_6.25u -> PCM_marbastlib-mx:STAB_MX_6.25u
- SW1, SW10, SW11, SW12, SW13, SW14, SW15, SW16, SW17, SW18, SW19, SW2, SW20, SW21, SW22, SW23, SW24, SW25, SW26, SW27, SW28, SW29, SW3, SW30, SW31, SW32, SW33, SW34, SW35, SW36, SW37, SW38, SW39, SW4, SW40, SW41, SW42, SW43, SW44, SW45, SW46, SW47, SW48, SW49, SW5, SW50, SW51, SW52, SW53, SW54, SW55, SW56, SW57, SW58, SW59, SW6, SW60, SW61, SW62, SW63, SW64, SW65, SW66, SW67, SW68, SW69, SW7, SW70, SW71, SW72, SW73, SW74, SW75, SW76, SW77, SW78, SW79, SW8, SW80, SW81, SW9: footprint (none) -> PCM_marbastlib-mx:SW_MX_1u
- SW82: footprint (none) -> PCM_marbastlib-various:ROT_Alps_EC11E-Switch
Other:
- moved on the sheet: A1, C1, C2, C3, D1, D10, D11, D12, D13, D14, D15, D16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
