File: FREEPCB/FREEBOARD.kicad_pcb (KiCad board)
At the start: 2 copper layers, 311.1 x 241.5 mm, 372 parts, among them J1 OLED_DISPLAY, SW1 SW_Push_45deg, SW10 SW_Push_45deg, SW11 SW_Push_45deg, SW12 SW_Push_45deg, SW13 SW_Push_45deg, SW14 SW_Push_45deg, SW15 SW_Push_45deg, SW16 SW_Push_45deg, SW17 SW_Push_45deg, SW18 SW_Push_45deg, SW19 SW_Push_45deg, SW2 SW_Push_45deg, SW20 SW_Push_45deg, SW21 SW_Push_45deg, SW22 SW_Push_45deg, SW23 SW_Push_45deg, SW24 SW_Push_45deg, SW25 SW_Push_45deg, SW26 SW_Push_45deg, SW27 SW_Push_45deg, SW28 SW_Push_45deg, SW29 SW_Push_45deg, SW3 SW_Push_45deg, SW30 SW_Push_45deg, SW31 SW_Push_45deg, SW32 SW_Push_45deg, SW33 SW_Push_45deg, SW34 SW_Push_45deg, SW35 SW_Push_45deg, SW36 SW_Push_45deg, SW37 SW_Push_45deg, SW38 SW_Push_45deg, SW39 SW_Push_45deg, SW4 SW_Push_45deg, SW40 SW_Push_45deg, SW41 SW_Push_45deg, SW42 SW_Push_45deg, SW43 SW_Push_45deg, SW44 SW_Push_45deg, SW45 SW_Push_45deg, SW46 SW_Push_45deg, SW47 SW_Push_45deg, SW48 SW_Push_45deg, SW49 SW_Push_45deg, SW5 SW_Push_45deg, SW50 SW_Push_45deg, SW51 SW_Push_45deg, SW52 SW_Push_45deg, SW53 SW_Push_45deg, SW54 SW_Push_45deg, SW55 SW_Push_45deg, SW56 SW_Push_45deg, SW57 SW_Push_45deg, SW58 SW_Push_45deg, SW59 SW_Push_45deg, SW6 SW_Push_45deg, SW60 SW_Push_45deg, SW61 SW_Push_45deg, SW62 SW_Push_45deg, SW63 SW_Push_45deg, SW64 SW_Push_45deg, SW65 SW_Push_45deg, SW66 SW_Push_45deg, SW67 SW_Push_45deg, SW68 SW_Push_45deg, SW69 SW_Push_45deg, SW7 SW_Push_45deg, SW70 SW_Push_45deg, SW71 SW_Push_45deg, SW72 SW_Push_45deg, SW73 SW_Push_45deg, SW74 SW_Push_45deg, SW75 SW_Push_45deg, SW76 SW_Push_45deg, SW77 SW_Push_45deg, SW78 SW_Push_45deg, SW79 SW_Push_45deg, SW8 SW_Push_45deg, SW80 SW_Push_45deg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

Commit message: PCB Update
Parts:
- C1: moved to B.Cu
- moved R2 308.0 mm to (315.8, 35.9), turned to 0 degrees
- moved R3 307.0 mm to (315.8, 33.5), turned to 0 degrees
- moved H1 305.4 mm to (41.9, 21.6)
- moved H5 287.5 mm to (39.5, 114.5)
- moved D1 285.8 mm to (56.2, 57.8)
- moved D14 285.8 mm to (341.9, 57.8)
- moved D15 285.8 mm to (56.2, 81.6)
- moved D29 285.8 mm to (341.9, 81.6)
- moved D44 285.8 mm to (341.9, 100.6)
- moved D58 285.8 mm to (341.9, 119.7)
- moved D72 285.8 mm to (341.9, 138.7)
- moved D81 285.8 mm to (341.9, 157.8)
- moved D73 281.0 mm to (58.6, 157.8)
- moved D30 276.2 mm to (61.0, 100.6)
- moved D45 271.5 mm to (63.3, 119.7)
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- renumbered D139 to D137, D142 to D138, D145 to D139, D148 to D140, D151 to D141, D154 to D142, D157 to D143, D160 to D144, D137 to D145, D140 to D146, D143 to D147, D146 to D148, D152 to D150, D155 to D151, D158 to D152, D161 to D153, D138 to D154, D141 to D155, D144 to D156, D147 to D157, D150 to D158, D153 to D159, D156 to D160, D159 to D161
Connections:
- J1 pad 1: /OLED_SDA -> GND
- J1 pad 2: /OLED_SCL -> /+5V
- J1 pad 3: /+5V -> /OLED_SCL
- J1 pad 4: GND -> /OLED_SDA
Routing:
- net /+5V: track 0.00 -> 2928.7 mm, vias 0 -> 127
- net /Row5: track 0.00 -> 563.2 mm, vias 0 -> 10
- net /Row4: track 0.00 -> 535.2 mm, vias 0 -> 4
- net /Row3: track 0.00 -> 513.2 mm, vias 0 -> 4
- net /Row2: track 0.00 -> 496.2 mm, vias 0 -> 5
- net /Row1: track 0.00 -> 473.3 mm, vias 0 -> 3
- net Net-(D162-DOUT): track 0.00 -> 469.9 mm
- net /Row0: track 0.00 -> 407.5 mm, vias 0 -> 1
- net Net-(D95-DOUT): track 0.00 -> 335.5 mm
- net Net-(D153-DOUT): track 0.00 -> 334.6 mm
- net /Col12: track 0.00 -> 332.4 mm
- net Net-(D110-DOUT): track 0.00 -> 324.3 mm
- net Net-(D125-DOUT): track 0.00 -> 324.2 mm
- net Net-(D139-DOUT): track 0.00 -> 319.1 mm
- net /Col13: track 0.00 -> 298.2 mm
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Other:
- board size 311.1 x 241.5 mm -> 311.1 x 246.3 mm

Commit message: PCB Update
Routing:
- net /+3V3: track 93.8 -> 212.3 mm, vias 4 -> 5
- net /Col3: track 172.0 -> 267.6 mm, vias 0 -> 2
- net /+5V: track 2928.7 -> 2984.4 mm, vias 127 -> 128
Other:
- board size 311.1 x 246.3 mm -> 311.1 x 248.7 mm

Commit message: PCB Update
Parts:
- removed C96: 100nF, Capacitor_SMD:C_0603_1608Metric_Pad1.08x0.95mm_HandSolder
- removed D173: SK6812MINI-E, footprints:SK6812MINI-E_fixed
- J1: footprint KiCad-SSD1306-0.91-OLED-4pin-128x32.pretty-master:SSD1306-0.91-OLED-4pin-128x32 -> Connector_JST:JST_SH_BM04B-SRSS-TB_1x04-1MP_P1.00mm_Vertical
- moved G*** 344.0 mm to (522.9, 162.1)
- moved G*** 344.0 mm to (523.2, 181.1)
- moved J1 29.6 mm to (304.2, 32.0), turned to 90 degrees
- turned C10 to 180 degrees
Connections:
- D172 pad 2: Net-(D172-DOUT) -> unconnected-(D172-DOUT-Pad2)
Routing:
- net GND: track 17.6 -> 1903.2 mm, vias 2 -> 169
- net Net-(D172-DOUT): track 72.9 -> 0.00 mm
- net /+5V: track 2984.4 -> 2965.3 mm, vias 128 -> 130
- net /OLED_SDA: track 135.0 -> 143.8 mm, vias 4 -> 5
- net /OLED_SCL: track 138.6 -> 145.7 mm, vias 4 -> 6
- net /ENC_A: track 102.2 -> 105.6 mm
- net /Row1: track 473.3 -> 474.8 mm
Other:
- board size 311.1 x 248.7 mm -> 314.3 x 164.3 mm

Commit message: PCB Complete
Parts:
- removed the G*** at (522.9, 162.1)
- removed the G*** at (523.2, 181.1)
- added G***: LOGO, LOGO, B.Cu at (210.2, 163.0)
- added G***: LOGO, LOGO, B.Cu at (210.2, 174.9)
- moved C36 63.8 mm to (71.8, 166.1)
- moved C37 63.8 mm to (95.6, 166.1)
- moved C38 63.8 mm to (114.7, 166.1)
- moved C39 63.8 mm to (133.7, 166.1)
- moved C40 63.8 mm to (152.8, 166.1)
- moved C41 63.8 mm to (171.8, 166.1)
- moved C42 63.8 mm to (190.9, 166.1)
- moved C43 63.8 mm to (209.9, 166.1)
- moved C44 63.8 mm to (229.0, 166.1)
- moved C45 63.8 mm to (248.0, 166.1)
- moved C46 63.8 mm to (267.1, 166.1)
- moved C47 63.8 mm to (286.1, 166.1)
- moved C65 63.8 mm to (79.0, 204.2)
- moved C66 63.8 mm to (109.9, 204.2)
- moved C67 63.8 mm to (129.0, 204.2)
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Routing:
- net GND: track 1903.2 -> 3329.9 mm, vias 169 -> 251
- net Net-(D153-DOUT): track 334.6 -> 333.2 mm
- net /+5V: track 2965.3 -> 2964.4 mm
Other:
- board size 314.3 x 164.3 mm -> 314.3 x 161.9 mm

Commit message: PCB Update
Parts:
- moved G*** 93.1 mm to (209.8, 81.8), turned to 0 degrees
- moved G*** 69.3 mm to (209.6, 93.7), turned to 0 degrees
